Commit message: hand core + retargeter interface, 47 tests passing

File: dataset/robot/l21_left/linkerhand_l21_left.urdf (robot description, URDF)
Before this commit: robot linkerhand_l21_left, 18 links, 17 joints
Links:
- added link index_tip, mass 0.001
- added link middle_tip, mass 0.001
- added link pinky_tip, mass 0.001
- added link ring_tip, mass 0.001
- added link thumb_tip, mass 0.001
Joints:
- added joint index_tip: type fixed, parent index_middle, child index_tip, origin xyz=0 0 0.044 rpy=0 0 0
- added joint middle_tip: type fixed, parent middle_middle, child middle_tip, origin xyz=0 0 0.044 rpy=0 0 0
- added joint pinky_tip: type fixed, parent pinky_middle, child pinky_tip, origin xyz=0 0 0.040 rpy=0 0 0
- added joint ring_tip: type fixed, parent ring_middle, child ring_tip, origin xyz=0 0 0.044 rpy=0 0 0
- added joint thumb_tip: type fixed, parent thumb_distal, child thumb_tip, origin xyz=0.026 0 0 rpy=0 0 0
